File: hw/balsamic/balsamic.sch (KiCad schematic (older format))
At the start: 4 parts, among them J1 Conn_01x24, U1 ISP1807-LR-RS, U2 BMI160, U3 K210

Commit message: Add hardware files
Parts:
- added J2: USB_C_Receptacle_USB2.0, Connector_USB:USB_C_Receptacle_XKB_U262-16XN-4BVC11, symbol Connector:USB_C_Receptacle_USB2.0
- added U4: CH552T, Package_SO:TSSOP-20_4.4x6.5mm_P0.65mm, symbol ch552t:CH552T
- added U5: GD25LQ, footprints:SOIC127P790X216-8N, symbol GD25LQ64:GD25LQ
Connections:
- new net: J2.A1 (GND), J2.A12 (GND), J2.B1 (GND), J2.B12 (GND)
- new net: J2.A4 (VBUS), J2.A9 (VBUS), J2.B4 (VBUS), J2.B9 (VBUS)
Other:
- moved on the sheet: U3A
Changed lines of the file:
@@
 L kendryte:K210 U3
 U 1 1 63572052
-P 2450 2300
-F 0 "U3" H 2175 3015 50  0000 C CNN
-F 1 "K210" H 2175 2924 50  0000 C CNN
-F 2 "footprints:Kendryte_K210" H 2200 2900 50  0001 C CNN
-F 3 "" H 2200 2900 50  0001 C CNN
-	1    2450 2300
+P 2150 3500
+F 0 "U3" H 1875 4215 50  0000 C CNN
+F 1 "K210" H 1875 4124 50  0000 C CNN
+F 2 "footprints:Kendryte_K210" H 1900 4100 50  0001 C CNN
+F 3 "" H 1900 4100 50  0001 C CNN
+	1    2150 3500
 	1    0    0    -1
 $EndComp
@@
 	1    0    0    -1
 $EndComp
+$Comp
+L ch552t:CH552T U4
+U 1 1 635F81A0
+P 6600 2850
+F 0 "U4" H 6600 3165 50  0000 C CNN
+F 1 "CH552T" H 6600 3074 50  0000 C CNN
+F 2 "Package_SO:TSSOP-20_4.4x6.5mm_P0.65mm" H 6600 2850 50  0001 C CNN
+F 3 "https://cdn.hackaday.io/files/1696717259204064/CH552%20Datasheet_C111367.zh-CN.en.pdf" H 6600 2850 50  0001 C CNN
+	1    6600 2850
+	1    0    0    -1
+$EndComp
+$Comp
+L Connector:USB_C_Receptacle_USB2.0 J2
+U 1 1 63606FA1
+P 1300 1500
+F 0 "J2" H 1407 2367 50  0000 C CNN
+F 1 "USB_C_Receptacle_USB2.0" H 1407 2276 50  0000 C CNN
+F 2 "Connector_USB:USB_C_Receptacle_XKB_U262-16XN-4BVC11" H 1450 1500 50  0001 C CNN
+F 3 "https://www.usb.org/sites/default/files/documents/usb_type-c.zip" H 1450 1500 50  0001 C CNN
+	1    1300 1500
+	1    0    0    -1
+$EndComp
+$Comp
+L GD25LQ64:GD25LQ U5
+U 1 1 635A09DA
+P 3850 7250
+F 0 "U5" H 3825 7715 50  0000 C CNN
+F 1 "GD25LQ" H 3825 7624 50  0000 C CNN
+F 2 "footprints:SOIC127P790X216-8N" H 3850 7250 50  0001 C CNN
+F 3 "https://www.digikey.com/en/products/detail/gigadevice-semiconductor-hk-limited/GD25LQ64CSIGR/9484705" H 3850 7250 50  0001 C CNN
+	1    3850 7250
+	1    0    0    -1
+$EndComp
