File: hw/balsamic/balsamic.kicad_sch (KiCad schematic)
At the start: 64 parts, among them J1 Conn_01x24, J2 USB_C_Receptacle_USB2.0, U1 ISP1807-LR-RS, U2 BMI160, U3 K210, U4 CH552T, U5 GD25LQ

Commit message: Schematic layout v0.1
Parts:
- removed C? (x2): 4.7pF, symbol Device:C_Small
- removed R?: 10k, symbol Device:R_Small
- removed SW?: SW_DIP_x02, symbol Switch:SW_DIP_x02
- removed Y?: Crystal_GND24, symbol Device:Crystal_GND24
- added BT?: Battery_Cell, symbol Device:Battery_Cell
- added C? (x4): 10uF, symbol Device:C_Small
- added C? (x2): 18pF, symbol Device:C_Small
- added C? (x2): 4.7pF, symbol Device:C_Small
- added C? (x2): 100nF, symbol Device:C_Small
- added C?: 22uF, symbol Device:C_Small
- added R? (x4): 100k, symbol Device:R_Small
- added R? (x2): 5.1k, symbol Device:R_Small
- added SW?: SW_Push_DPDT, symbol Switch:SW_Push_DPDT
- added Y? (x2): Crystal_GND24, symbol Device:Crystal_GND24
Connections:
- net DC Charging Input is gone; now on net VBUS: C?.1, U?.A1 (CHGIN)
- net RESET is gone; now on net CH552_P1.0: U3.M1 (RESETN)
- net +1V8: now also J1.11 (Pin_11), R?.1, R?.2
- net +3V3: now also J1.10 (Pin_10), C?.1, R?.1
- net BATT: now also BT?.1 (+)
- net BOOT: no longer R?.2
- net DVP_D0: now also J1.19 (Pin_19)
- net DVP_D1: now also J1.21 (Pin_21)
- net DVP_D2: now also J1.22 (Pin_22)
- net DVP_D3: now also J1.20 (Pin_20)
- net DVP_D4: now also J1.18 (Pin_18)
- net DVP_D5: now also J1.16 (Pin_16)
- net DVP_D6: now also J1.14 (Pin_14)
- net DVP_D7: now also J1.12 (Pin_12)
- net DVP_HSYNC: now also J1.9 (Pin_9)
- net DVP_PCLK: now also J1.17 (Pin_17)
- net DVP_PWDN: now also J1.8 (Pin_8)
- net DVP_RST: now also J1.6 (Pin_6)
- net DVP_SCL: now also J1.5 (Pin_5), R?.2
- net DVP_SDA: now also J1.3 (Pin_3), R?.1
- net DVP_VSYNC: now also J1.7 (Pin_7)
- net DVP_XCLK: now also J1.13 (Pin_13)
- net GND: now also J1.15 (Pin_15), J2.A1 (GND), J2.A12 (GND), J2.B1 (GND), J2.B12 (GND), J2.S1 (SHIELD), U2.6 (GNDIO), U2.7 (GND), U4.18 (GND), BT?.2 (-), C?.1, C?.1, C?.1, C?.1, C?.2, C?.2, C?.2, C?.2, R?.2, R?.2, R?.2, Y?.2, Y?.2, Y?.4, Y?.4
- net IO_6: no longer SW?.1
- net LDO_0: now also U1.26 (VCC_NRF)
- net LDO_1: now also J1.4 (Pin_4), U2.5 (VDDIO), U2.8 (VDD), C?.1, C?.1, C?.1, C?.2, C?.2
- net SPI_CLK: now also U1.32 (P0_08), U2.13 (SCx)
- net VBUS: now also J2.A4 (VBUS), J2.A9 (VBUS), J2.B4 (VBUS), J2.B9 (VBUS), U4.19 (VCC)
- net SPI_MISO: now reaches U2.1 (SDO)
- net SPI_MISO: now also U1.35 (P0_04_AIN2)
- net SPI_CS_IMU: now reaches U2.12 (CSB)
- net SPI_CS_IMU: now also U1.33 (P0_07_TRACECLK)
- net SPI_MOSI: now reaches U2.14 (SDx)
- net SPI_MOSI: now also U1.34 (P0_06)
- net INT_1_IMU: now reaches U2.4 (INT1)
- net INT_2_IMU: now reaches U2.9 (INT2)
- net X_OUT_K210: now reaches R?.1, U3.M3 (OSC_26M_XOUT)
- net X_OUT_K210: now also C?.2, Y?.3
- net X_IN_K210: now reaches R?.2, U3.M4 (OSC_26M_XIN)
- net X_IN_K210: now also C?.1, Y?.1
- net UART_RX_nRF: now reaches U3.A12 (IO_17)
- net UART_RX_nRF: now also U1.37 (P0_15)
- net UART_TX_nRF: now reaches U3.C12 (IO_15)
- net UART_TX_nRF: now also U1.36 (P0_05_AIN3)
- net Button: now reaches U1.39 (P0_27)
- net Button: now also SW?.1
- net GNDA: now reaches J1.2 (Pin_2)
- net GNDA: now also C?.2, C?.2, C?.2
- net at J1.23 (Pin_23): now also R?.2
- net at J1.24 (Pin_24): now also R?.1
- net USB_D+_K210: now reaches U4.14 (P3.6)
- net USB_D+_K210: now also SW?.6 (C)
- net USB_D-_K210: now reaches U4.15 (P3.7)
- net USB_D-_K210: now also SW?.3 (C)
- net X_OUT_CH552: now reaches U4.16 (P1.3)
- net X_OUT_CH552: now also C?.2, Y?.3
- net X_IN_CH552: now reaches U4.17 (P1.2)
- net X_IN_CH552: now also C?.1, Y?.1
- net at U4.20 (V33): now also C?.1
- net at J2.A5 (CC1): now also R?.1
- net USB_D+: now reaches J2.A6 (D+)
- net USB_D+: now also J2.B6 (D+), SW?.5 (B)
- net USB_D-: now reaches J2.A7 (D-)
- net USB_D-: now also J2.B7 (D-), SW?.2 (B)
- net at J2.B5 (CC2): now also R?.1
- net CH552_P1.1 renamed BOOT_K210
- net BOOT_K210: now also R?.2
- net OSC_CLK renamed 26M_OUT_K210
- net SPIO_CS0: no longer names the net of U3.A6 (IO_29)
- net SPIO_MISO: no longer names the net of U3.B7 (IO_26)
- net SPIO_MOSI: no longer names the net of U3.B6 (IO_28)
- net SPIO_SCLK: no longer names the net of U3.A7 (IO_27)
- net SWDCLK renamed SWDCLK_nRF
- net SWDCLK_nRF: now also SW?.4 (A)
- net SWDIO renamed SWDIO_nRF
- net SWDIO_nRF: now also SW?.1 (A)
- no-connect marks 104 -> 107
Other:
- note added: "24MHz 12 pF 10ppm"
- note added: "Battery"
- note added: "Button"
- note added: "Camera"
- note added: "Camera Analog Power"
- note added: "Camera Digital Power"
- note added: "Flash"
- note added: "IMU"
- note added: "ISP1807"
- note added: "Input Power from Max"
- note added: "Input Power from USB"
- note added: "Internal Pullup on nRF; trigger interrupt to wake nRF"
- note added: "Kendryte Programming"
- note added: "To Kendryte K210"
- note added: "Toggle between programming K210 and ISP1807"
- note added: "Will need separate analog and ground planes"
- note removed: "ISP Download"
- note removed: "User Interactive Button"
- moved on the sheet: C?, J1, J2, R?, SW?, U1, U2, U3D, U3G, U3H, U4, U5

Commit message: Removed CH552T for programming
Parts:
- removed C? (x12): 100nF, symbol Device:C_Small
- removed C?: 1uF, symbol Device:C_Small
- removed C? (x2): 18pF, symbol Device:C_Small
- removed C? (x2): 10uF, symbol Device:C_Small
- removed C? (x3): 22uF, symbol Device:C_Small
- removed J2: USB_C_Receptacle_USB2.0, Connector_USB:USB_C_Receptacle_XKB_U262-16XN-4BVC11, symbol balsamic-rescue:USB_C_Receptacle_USB2.0-Connector
- removed R? (x2): 5.1k, symbol Device:R_Small
- removed R?: 10k, symbol Device:R_Small
- removed R?: 100k, symbol Device:R_Small
- removed SW?: SW_Push_DPDT, symbol Switch:SW_Push_DPDT
- removed U4: CH552T, Package_SO:TSSOP-20_4.4x6.5mm_P0.65mm, symbol balsamic-rescue:CH552T-ch552t
- removed Y?: Crystal_GND24, symbol Device:Crystal_GND24
- added C? (x5): 10uF, symbol Device:C_Small
- added C? (x5): 100uF, symbol Device:C_Small
- added C? (x4): 4.7uF, symbol Device:C_Small
- added C? (x3): 22uF, symbol Device:C_Small
- added C?: 1uF, symbol Device:C_Small
- added C?: 100nF, symbol Device:C_Small
- added C?: 100nf, symbol Device:C_Small
- added D? (x2): LED, symbol Device:LED
- added J?: USB_C_Receptacle, symbol Connector:USB_C_Receptacle
- added R? (x2): 4.7K, symbol Device:R_Small
- added R? (x2): 200, symbol Device:R_Small
- added R? (x2): 5.1k, symbol Device:R_Small
- added R? (x3): 0, symbol Device:R_Small
- added TP? (x15): TestPoint, symbol Connector:TestPoint
- R? (x2): value 100k -> 10k
- R? (x2): value 100k -> 0
Connections:
- net ALRT is gone; now on net PMU_ALERT_PIN: U?.B5 (ALRT)
- net BOOT is gone; now on net BOOT_K210: U3.B12 (IO_16)
- net SCL is gone; now on net PMU_SCL: U?.B4 (SCL)
- net SDA is gone; now on net PMU_SDA: U?.C4 (SDA)
- net SWDCLK_nRF is gone; now on net USB_D+: U1.30 (SWDCLK)
- net SWDIO_nRF is gone; now on net USB_D-: U1.28 (SWDIO)
- net +0V9: now also C?.1, TP?.1
- net +1V8: now also C?.1, J1.10 (Pin_10), U1.26 (VCC_NRF), U2.5 (VDDIO), U2.8 (VDD), U3.D3 (VDDIO33_3), U3.F3 (VDDIO33_5), U3.G10 (VDDIO33_6), U5.8 (VCC), C?.1, C?.1, C?.2, C?.2, TP?.1
- net +3V3: now also C?.1, TP?.1; no longer C?.1, J1.10 (Pin_10), U3.D3 (VDDIO33_3), U3.F3 (VDDIO33_5), U3.G10 (VDDIO33_6)
- net BATT: now also C?.1, C?.1, C?.1, C?.1, C?.1, C?.1, C?.1, C?.1, C?.1, C?.1, C?.1, C?.1, C?.1, C?.1, R?.2; no longer U?.A4 (TH)
- net BOOT_K210: no longer R?.2
- net CH552_P1.0: now also J?.A11 (RX2+), J?.B11 (RX1+)
- net CH552_RX0: now also J?.A10 (RX2-), J?.B10 (RX1-)
- net CH552_TX0: now also J?.A3 (TX1-), J?.B3 (TX2-)
- net DVP_SCL: now also TP?.1
- net DVP_SDA: now also TP?.1
- net F_CS: now also U5.1 (CS)
- net F_D0: now also U5.5 (SI/IO0)
- net F_D1: now also U5.2 (SO/IO1)
- net F_D2: now also U5.3 (WP/IO2)
- net F_D3: now also U5.7 (HOLD/IO3)
- net GND: now also U5.4 (GND), C?.1, C?.1, C?.2, C?.2, C?.2, C?.2, C?.2, C?.2, C?.2, C?.2, C?.2, C?.2, C?.2, C?.2, C?.2, C?.2, C?.2, C?.2, C?.2, C?.2, D?.1 (K), D?.1 (K), J?.A1 (GND), J?.A12 (GND), J?.B1 (GND), J?.B12 (GND), J?.S1 (SHIELD), R?.2, R?.2
- net GNDA: now also C?.1; no longer C?.2
- net INT_1_IMU: now also U1.61 (P1_11), TP?.1
- net INT_2_IMU: now also U1.60 (P1_10), TP?.1
- net LDO_1: no longer C?.1, C?.1, C?.2, C?.2, J1.4 (Pin_4), R?.1, U2.5 (VDDIO), U2.8 (VDD)
- net NIRQ: now also U1.62 (P1_07)
- net SPI_CLK: no longer U3.K1 (SPI_CLK)
- net USB_D+: now also J?.A6 (D+), J?.B6 (D+), TP?.1
- net USB_D-: now also J?.A7 (D-), J?.B7 (D-), TP?.1
- net at U3.A1 (IO_37): now also R?.1
- net at U3.A2 (IO_36): now also R?.2
- net nRF_UART_RX: now reaches U3.G12 (IO_7)
- net nRF_UART_RX: now also U1.37 (P0_15), R?.1, TP?.1
- net F_CLK: now reaches U5.6 (CLK)
- net F_CLK: now also U3.K1 (SPI_CLK)
- net nRF_UART_RX_DBUG: now reaches U1.41 (P0_25)
- net nRF_UART_RX_DBUG: now also TP?.1
- net nRF_UART_TX_DBUG: now reaches U1.43 (P0_11_TRACEDATA)
- net nRF_UART_TX_DBUG: now also TP?.1
- net PMU_SCL: now reaches U1.56 (P1_09_TRACEDATA3)
- net PMU_SCL: now also R?.2
- net PMU_SDA: now reaches U1.57 (P1_00_TRACEDATA0)
- net PMU_SDA: now also R?.2
- net nRF_GPIO_1: now reaches U1.58 (P1_03)
- net nRF_GPIO_1: now also R?.2
- net nRF_GPIO_0: now reaches U1.59 (P1_12)
- net nRF_GPIO_0: now also R?.2
- net PMU_ALERT_PIN: now reaches U1.63 (P1_04)
- net VSYS: now reaches C?.1, U?.A2 (SYS), U?.D6 (IN_SBB)
- net VSYS: now also R?.1; no longer U?.D1 (NEN)
- net GPIO_0 renamed PMU_GPIO_0
- net GPIO_1 renamed PMU_GPIO_1
- net GPIO_2 renamed PMU_GPIO_2
- net IO_6 renamed nRF_UART_TX
- net nRF_UART_TX: now also U1.36 (P0_05_AIN3), R?.2, TP?.1
- net JTAG_TID renamed JTAG_TDI
- net LDO_0 renamed +3V0
- net +3V0: now also C?.1, C?.2, TP?.1; no longer U1.26 (VCC_NRF)
- net NRST: no longer names the net of U?.F3 (NRST)
- net RST_ISP renamed VCC
- net VCC: now also R?.1, R?.1
- net UART_RX_nRF: no longer names the net of U3.A12 (IO_17)
- net UART_RX_nRF: no longer U1.37 (P0_15)
- net UART_TX_nRF: no longer names the net of U3.C12 (IO_15)
- net UART_TX_nRF: no longer U1.36 (P0_05_AIN3)
- net VBUS renamed VBUS_USB
- net VBUS_USB: now also J?.A4 (VBUS), J?.A9 (VBUS), J?.B4 (VBUS), J?.B9 (VBUS)
- net X_IN_K210 renamed K210_X_IN
- net K210_X_IN: now also C?.2, Y?.3; no longer C?.1, Y?.1
- net X_OUT_K210 renamed K210_X_OUT
- net K210_X_OUT: now also C?.1, Y?.1; no longer C?.2, Y?.3
- new net: D?.2 (A), R?.1 (x2)
- new net: J?.B5 (CC2), R?.1
- new net: J?.A5 (CC1), R?.1
- new net: R?.1, U?.A4 (TH)
- new net CH552_P1.1: J?.A2 (TX1+), J?.B2 (TX2+), R?.2
- new net VDDA: C?.2, C?.2, J1.4 (Pin_4)
- new net nRF_GPIO: TP?.1
- no-connect marks 107 -> 90
Other:
- note added: "10V/(0201)"
- note added: "25V/(0201)"
- note added: "25V/(0402)"
- note added: "Camera control"
- note added: "Clock and Boot"
- note added: "During power-on reset, pull IO_16 high to boot from FLASH and pull low to enter ISP mode. (from K210 datasheet)"
- note added: "Flash control"
- note added: "I2C Pullups"
- note added: "SIMO (buck-boost) and LDO outputs from MAX"
- note added: "Status LEDs"
- note added: "Test Points"
- note added: "To nRF ISP1807"
- note added: "analog supply"
- note added: "nRF Ground Pins"
- note added: "nRF ISP1807"
- note added: "nRF Reset"
- note removed: "10V/(0603)"
- note removed: "24MHz 12 pF 10ppm"
- note removed: "25V/(0603)"
- note removed: "6.3V/(0603)"
- note removed: "ISP Power Ground Pins"
- note removed: "ISP Reset"
- note removed: "ISP1807"
- note removed: "Kendryte Programming"
- note removed: "Toggle between programming K210 and ISP1807"
- note removed: "dont forget to add pull ups for I2C"
- moved on the sheet: C?, J1, L?, R?, U1, U3B, U3C, U3D, U3E, U3F, U3G, U3H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

Commit message: Made some updates to schematic USB C and power
Parts:
- removed BT?: Battery_Cell, symbol Device:Battery_Cell
- removed D? (x2): LED, symbol Device:LED
- removed R? (x2): 200, symbol Device:R_Small
- removed TP?: TestPoint, symbol Connector:TestPoint
- added BT1: GREPOW_Battery, footprints:balsamic_grepow_battery, symbol kendryte-power:GREPOW_Battery
- added C51: 10uF, Capacitor_SMD:C_0402_1005Metric, symbol Device:C_Small
- added C52: 1uF, Capacitor_SMD:C_0402_1005Metric, symbol Device:C_Small
- added C53: 1uF, Capacitor_SMD:C_0201_0603Metric, symbol Device:C_Small
- added C54: 100nF, Capacitor_SMD:C_0402_1005Metric, symbol Device:C_Small
- added H1, H2, H3, H4: MountingHole_Pad, MountingHole:MountingHole_2.2mm_M2_DIN965_Pad, symbol Mechanical:MountingHole_Pad
- added R13, R14: 2k, Resistor_SMD:R_0201_0603Metric, symbol Device:R_Small
- added R19, R21: 100k, Resistor_SMD:R_0201_0603Metric, symbol Device:R_Small
- added R20: 0, Resistor_SMD:R_0201_0603Metric, symbol Device:R_Small
- added U6: MAX811LEUS-T, Package_TO_SOT_SMD:SOT-143, symbol Power_Supervisor:MAX811LEUS-T
- added U7: SiP32431DR3, Package_TO_SOT_SMD:SOT-363_SC-70-6, symbol Power_Management:SiP32431DR3
- C1, C10, C11, C12, C13, C14, C15, C16, C17, C18, C19, C2, C20, C21, C22, C24, C25, C26, C27, C29, C3, C30, C31, C32, C33, C35, C36, C37, C38, C4, C40, C41, C42, C43, C44, C45, C46, C47, C48, C49, C5, C6, C7, C8, C9: renamed from C?; footprint (none) -> Capacitor_SMD:C_0402_1005Metric
- C23, C28, C34, C39, C50: renamed from C?; footprint (none) -> Capacitor_SMD:C_0201_0603Metric
- FB1, FB2: renamed from FB?; footprint (none) -> Inductor_SMD:L_0603_1608Metric
- J2: renamed from J?; footprint (none) -> Connector_USB:USB_C_Receptacle_Amphenol_12401610E4-2A
- L1: renamed from L?; footprint (none) -> Inductor_SMD:L_0805_2012Metric
- R1, R10, R11, R12, R15, R16, R17, R18, R2, R3, R4, R5, R6, R7, R8, R9: renamed from R?; footprint (none) -> Resistor_SMD:R_0201_0603Metric
- SW1: renamed from SW?; footprint (none) -> Button_Switch_SMD:SW_SPST_B3U-1000P
- TP1, TP10, TP11, TP12, TP13, TP14, TP15, TP2, TP3, TP4, TP6, TP7, TP8, TP9: renamed from TP?; footprint (none) -> TestPoint:TestPoint_Pad_1.0x1.0mm
- U4: renamed from U?; footprint 21-100490_N362A3+1_MXM -> footprints:MAX77658AANX&plus_
- Y1: renamed from Y?; footprint (none) -> Crystal:Crystal_SMD_3225-4Pin_3.2x2.5mm
- gave numbers to parts that had none: 1
Connections:
- net LDO_1 is gone; now on net +1V8: U4.B3 (VIO), U4.E1 (LDO1)
- net +1V8: now also C52.2, C53.1, R13.1, R19.1; no longer C3.2, U2.5 (VDDIO), U2.8 (VDD), U5.8 (VCC)
- net +3V0: now also J1.4 (Pin_4)
- net +3V3: now also U6.4 (VCC)
- net BATT: now also BT1.1 (+)
- net CH552_P1.0: now also C51.1, R19.2, U6.2 (~{RESET})
- net GND: now also BT1.2 (-), C51.2, C52.1, C53.2, C54.1, H1.1, H2.1, H3.1, H4.1, U6.1 (GND), U7.2 (GND), U7.5 (GND)
- net VCC: now also R21.2; no longer U1.13 (P0_18_RESET)
- net VDD_nRF: now reaches U1.55 (P1_08)
- net VDD_nRF: now also C45.2, C46.2, R20.1
- net SBU1: now reaches J2.A8 (SBU1)
- net SBU1: now also J2.B8 (SBU2), U1.13 (P0_18_RESET), C54.2, R21.1
- removed net VDDA: C45.2, C46.2, J1.4 (Pin_4)
- net nRF_GPIO_0: no longer names the net of U1.59 (P1_12)
- net nRF_GPIO_1: no longer names the net of U1.58 (P1_03)
- new net: R20.2, U2.5 (VDDIO), U2.8 (VDD)
- new net: C3.2, R14.2, U5.8 (VCC), U7.1 (OUT)
- new net: R13.2, R14.1, U7.4 (IN)
- new net FLASH_EN: U7.3 (ON)
- no-connect marks 90 -> 91
Other:
- note added: "Load Switch"
- note added: "Mount Hole"
- note added: "Power On Reset"
- note added: "digital supply"
- note added: "pull IO_16 high to boot FLASH and pull low to enter ISP mode."
- note removed: "During power-on reset, pull IO_16 high to boot from FLASH and pull low to enter ISP mode. (from K210 datasheet)"
- note removed: "Status LEDs"
- moved on the sheet: C1, C2, C3, C45, C46, C47, C48, C49, C50, J1, J2, R1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

Commit message: Began board Layout
Parts:
- removed C54: 100nF, Capacitor_SMD:C_0402_1005Metric, symbol Device:C_Small
- removed H1, H2, H3, H4: MountingHole_Pad, MountingHole:MountingHole_2.2mm_M2_DIN965_Pad, symbol Mechanical:MountingHole_Pad
- added D1, D2: LED, LED_SMD:LED_0402_1005Metric, symbol Device:LED
- added R22, R23, R24, R25, R26, R27, R28, R29, R30, R31, R32, R35: 0, Resistor_SMD:R_0402_1005Metric, symbol Device:R_Small
- added R33, R34: 220, Resistor_SMD:R_0201_0603Metric, symbol Device:R_Small
- added TP16, TP17, TP18, TP19, TP20, TP5: TestPoint, TestPoint:TestPoint_Pad_1.0x1.0mm, symbol Connector:TestPoint
- C1, C13, C2: footprint Capacitor_SMD:C_0402_1005Metric -> Capacitor_SMD:C_0201_0603Metric
- FB1, FB2: footprint Inductor_SMD:L_0603_1608Metric -> Inductor_SMD:L_0201_0603Metric
- R13: value 2k -> 0
- R14: value 2k -> NO_STUFF
- R15, R16: value 10k -> 4.7K
- R20: value 0 -> NO_STUFF
- R21: value 100k -> 0; footprint Resistor_SMD:R_0201_0603Metric -> Resistor_SMD:R_0402_1005Metric
Connections:
- net +1V8: now also R20.1; no longer C14.1, U3.D3 (VDDIO33_3), U3.F3 (VDDIO33_5), U3.G10 (VDDIO33_6), U3.H3 (VDDIO18_0), U3.J3 (VDDOTP), U3.K6 (VDDIO18_1), U3.K8 (VDDIO18_2)
- net +3V0: now also D1.2 (A), D2.2 (A)
- net BATT: now also R35.2; no longer BT1.1 (+)
- net CH552_P1.0: now also R26.2, R30.2; no longer J2.A11 (RX2+), J2.B11 (RX1+)
- net CH552_P1.1: now also R28.2, R32.2; no longer J2.A2 (TX1+), J2.B2 (TX2+)
- net CH552_RX0: now also R25.2, R29.2; no longer J2.A10 (RX2-), J2.B10 (RX1-)
- net CH552_TX0: now also R27.2, R31.2; no longer J2.A3 (TX1-), J2.B3 (TX2-)
- net NIRQ: now also TP5.1
- net PMU_ALERT_PIN: now also TP16.1
- net SPI_CLK: now also TP19.1
- net SPI_CS_IMU: now also TP20.1
- net SPI_MISO: now also TP17.1
- net SPI_MOSI: now also TP18.1
- net USB_D+: now also R23.2, R24.2; no longer J2.A6 (D+), J2.B6 (D+)
- net USB_D-: now also R21.2, R22.2; no longer J2.A7 (D-), J2.B7 (D-)
- net VCC: no longer R21.2
- net VDD_nRF: now also R20.2, U2.5 (VDDIO), U2.8 (VDD); no longer R20.1
- net nRF_UART_RX: no longer U3.G12 (IO_7)
- net nRF_UART_TX: no longer U3.G11 (IO_6)
- net nRF_UART_TX_DBUG: now also J2.A8 (SBU1), J2.B8 (SBU2)
- net K210_1V8: now reaches C3.2, R14.2, U5.8 (VCC), U7.1 (OUT)
- net K210_1V8: now also C14.1, U3.D3 (VDDIO33_3), U3.F3 (VDDIO33_5), U3.G10 (VDDIO33_6), U3.H3 (VDDIO18_0), U3.J3 (VDDOTP), U3.K6 (VDDIO18_1), U3.K8 (VDDIO18_2)
- net nRF_LED2: now reaches U1.58 (P1_03)
- net nRF_LED2: now also R34.1
- net nRF_LED1: now reaches U1.59 (P1_12)
- net nRF_LED1: now also R33.1
- removed net SBU1: J2.A8 (SBU1), J2.B8 (SBU2), R21.1, U1.13 (P0_18_RESET)
- new net: J2.B3 (TX2-), R31.1
- new net: BT1.1 (+), R35.1
- new net: J2.A2 (TX1+), R28.1
- new net: J2.B2 (TX2+), R32.1
- new net: D2.1 (K), R34.2
- new net: J2.B10 (RX1-), R25.1
- new net: J2.B7 (D-), R22.1
- new net: J2.A11 (RX2+), R30.1
- new net: J2.B6 (D+), R24.1
- new net: J2.A10 (RX2-), R29.1
- new net: J2.A3 (TX1-), R27.1
- new net: J2.A6 (D+), R23.1
- new net: J2.A7 (D-), R21.1
- new net: J2.B11 (RX1+), R26.1
- new net: D1.1 (K), R33.2
- new net nRF_RST: U1.13 (P0_18_RESET)
Other:
- note added: "LEDs"
- note removed: "Mount Hole"
- note removed: "nRF Reset"
- moved on the sheet: BT1, C45, C46, J2, R11, R12, R20, R4, R5, TP10, TP11, TP12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

Commit message: Board layout v.1
Connections:
- net +1V8: no longer C33.1, C38.1
- net K210_1V8: now also C33.1, C38.1
Changed lines of the file:
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@@
     (stroke (width 0) (type default) (color 0 0 0 0))
   )
-  (wire (pts (xy 200.66 200.66) (xy 200.66 201.93))
-    (stroke (width 0) (type default) (color 0 0 0 0))
-  )
   (wire (pts (xy 227.33 97.79) (xy 229.87 97.79))
     (stroke (width 0) (type default) (color 0 0 0 0))
@@
     (stroke (width 0) (type default) (color 0 0 0 0))
   )
-  (polyline (pts (xy 270.51 121.92) (xy 420.37 123.19))
+  (polyline (pts (xy 270.51 123.19) (xy 420.37 123.19))
     (stroke (width 1) (type default) (color 0 0 0 0))
   )
@@
     )
   )
+  (global_label "K210_1V8" (shape input) (at 200.66 201.93 180) (fields_autoplaced)
+    (effects (font (size 1.27 1.27)) (justify right))
+    (property "Intersheet References" "${INTERSHEET_REFS}" (id 0) (at 188.962 202.0094 0)
+      (effects (font (size 1.27 1.27)) (justify right) hide)
+    )
+  )
   (global_label "F_D3" (shape input) (at 38.1 236.22 0) (fields_autoplaced)
     (effects (font (size 1.27 1.27)) (justify left))
@@
     (pin "1")
   )
-  (symbol (lib_id "power:+1V8") (at 200.66 200.66 0) (unit 1)
-    (in_bom yes) (on_board yes) (fields_autoplaced)
-    (property "Reference" "#PWR032" (id 0) (at 200.66 204.47 0)
-      (effects (font (size 1.27 1.27)) hide)
-    )
-    (property "Value" "+1V8" (id 1) (at 200.66 195.58 0))
-    (property "Footprint" "" (id 2) (at 200.66 200.66 0)
-      (effects (font (size 1.27 1.27)) hide)
-    )
-    (property "Datasheet" "" (id 3) (at 200.66 200.66 0)
-      (effects (font (size 1.27 1.27)) hide)
-    )
-    (pin "1")
-  )
   (symbol (lib_id "Device:C_Small") (at 207.01 74.93 180) (unit 1)
     (in_bom yes) (on_board yes)
@@
   (symbol (lib_id "Device:R_Small") (at 33.02 200.66 270) (unit 1)
     (in_bom yes) (on_board yes)
-    (property "Reference" "R3" (id 0) (at 33.9087 202.6325 90))
-    (property "Value" "0" (id 1) (at 31.7377 202.5705 90))
+    (property "Reference" "R3" (id 0) (at 31.75 203.2 90))
+    (property "Value" "0" (id 1) (at 34.29 203.2 90))
     (property "Footprint" "Resistor_SMD:R_0201_0603Metric" (id 2) (at 33.02 200.66 0)
       (effects (font (size 1.27 1.27)) hide)
@@
       (reference "#PWR031") (unit 1) (value "+3V3") (footprint "")
     )
-    (path "/215478ab-8ccf-4428-9102-ef89e0741243"
-      (reference "#PWR032") (unit 1) (value "+1V8") (footprint "")
-    )
     (path "/0185079a-0557-49b8-8c80-75e4a28f470e"

Commit message: Reduced spacing between ICs
Parts:
- removed R21, R24, R29, R30, R31, R32: 0, Resistor_SMD:R_0402_1005Metric, symbol Device:R_Small
- removed R4, R5: 5.1k, Resistor_SMD:R_0201_0603Metric, symbol Device:R_Small
- removed TP1, TP10, TP11, TP12, TP13, TP2, TP3, TP4, TP6, TP7, TP8, TP9: TestPoint, TestPoint:TestPoint_Pad_1.0x1.0mm, symbol Connector:TestPoint
- C10, C11, C12, C14, C15, C16, C17, C18, C19, C20, C21, C22, C24, C25, C26, C27, C29, C3, C30, C31, C32, C33, C35, C36, C37, C38, C4, C40, C41, C42, C43, C44, C45, C47, C48, C49, C5, C51, C52, C6, C7, C8, C9: footprint Capacitor_SMD:C_0402_1005Metric -> Capacitor_SMD:C_0201_0603Metric
- TP14, TP15, TP16, TP17, TP18, TP19, TP20, TP5: footprint TestPoint:TestPoint_Pad_1.0x1.0mm -> TestPoint:TestPoint_Pad_D1.0mm
Connections:
- net nRF_UART_RX_DBUG: now also J2.A5 (CC1), J2.B5 (CC2)
- net at J2.B3 (TX2-): now also J2.A3 (TX1-), R27.1
- net at J2.A2 (TX1+), R28.1: now also J2.B2 (TX2+)
- net at J2.B10 (RX1-), R25.1: now also J2.A10 (RX2-)
- net at J2.B7 (D-), R22.1: now also J2.A7 (D-)
- net at J2.A11 (RX2+): now also J2.B11 (RX1+), R26.1
- net at J2.B6 (D+): now also J2.A6 (D+), R23.1
- net JTAG_TCK: no longer names the net of U3.K11 (IO_0)
- net JTAG_TDI: no longer names the net of U3.K12 (IO_1)
- net JTAG_TDO: no longer names the net of U3.J12 (IO_3)
- net JTAG_TMS: no longer names the net of U3.J11 (IO_2)
- no-connect marks 91 -> 95
Other:
- moved on the sheet: R22, R27, R28, R7, R8
